File: hardware/radio_module/rev_a/radio_module.brd (EAGLE design)
At the start: 68.1 x 66 mm, 122 parts, among them J1 MODULE_GENERIC, J2 TC2030-JLINK-NL, J4 NANO_SIM, J5 TC2030-JLINK-L, P1 MOLEX_73251-135X, P2 MOLEX_73251-135X, Q1 MOSFET-NCHANNELXFDN-3, Q2 MOSFET-NCHANNELXFDN-3, Q3 MOSFET-NCHANNELXFDN-3, Q4 MOSFET-NCHANNELXFDN-3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

Commit message: made some changes...waiting on gthan
Parts:
- TP14, TP15, TP16, TP17: value PTR1PAD1-13 -> TEST_POINT_0.040IN; device testpad:P1-13 -> headers:TESTPOINT_0.040IN
- moved TP17 7.26 mm to (51.6, 60.2)
- moved R38 2.03 mm to (18.7, 53.6)
- moved R34 1.65 mm to (57.7, 49.3)
- moved C26 1.42 mm to (20.8, 61.3), turned to 270 degrees
- moved TP16 1.40 mm to (51.8, 66.5)
- moved Q3 1.20 mm to (24.9, 40.3)
- moved C11 1.17 mm to (9.78, 22.4)
- moved C2 1.14 mm to (46.9, 35.1)
- moved R32 1.02 mm to (6.48, 34.3)
- moved C12 0.97 mm to (54.0, 59.4)
- moved U8 0.90 mm to (22.9, 56.5)
- moved C20 0.89 mm to (25.3, 27.1)
- moved TP13 0.89 mm to (44.5, 47.5)
- moved TP5 0.89 mm to (46.2, 47.5)
- moved R25 0.81 mm to (24.9, 41.7)
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Connections:
- net 3V3: now also TP17.TESTPOINT; no longer TP17.TP
- net 3V8: now also TP14.TESTPOINT; no longer TP14.TP
- net 5V: now also TP16.TESTPOINT; no longer TP16.TP
- net GND: now also TP15.TESTPOINT; no longer TP15.TP
Routing:
- net USB_D-: track 50.0 -> 40.5 mm
- net N$15: track 32.7 -> 23.4 mm
- net USB_D+: track 53.1 -> 43.8 mm
- net GSM_LED: track 33.3 -> 24.4 mm
- net CONTROLLER_BUCK/LDO_N: track 27.0 -> 20.1 mm
- net GND: track 17.1 -> 11.4 mm, vias 170 -> 125
- net N$41: track 1.65 -> 5.27 mm
- net 3V8: track 25.5 -> 27.5 mm
- net GSM_3V8: track 58.8 -> 60.9 mm
- net GSM_POWER: track 9.91 -> 8.11 mm
- net N$16: track 2.66 -> 4.14 mm
- net NUCLEUM_GAUGE_ALERT: track 13.7 -> 15.1 mm
- net 5V: track 53.6 -> 52.2 mm
- net N$38: track 1.67 -> 2.95 mm
- net !GSM_RST: track 12.4 -> 11.3 mm
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