File: hardware/radio_module/rev_a/radio_module.sch (EAGLE design)
At the start: 122 parts, among them J1 MODULE_GENERIC, J2 TC2030-JLINK-NL, J4 NANO_SIM, J5 TC2030-JLINK-L, P1 MOLEX_73251-135X, P2 MOLEX_73251-135X, Q1 MOSFET-NCHANNELXFDN-3, Q2 MOSFET-NCHANNELXFDN-3, Q3 MOSFET-NCHANNELXFDN-3, Q4 MOSFET-NCHANNELXFDN-3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

Commit message: made some changes...waiting on gthan
Parts:
- TP14, TP15, TP16, TP17: value PTR1PAD1-13 -> TEST_POINT_0.040IN; device testpad:PTR1PAD1-13 -> headers:TEST_POINT_0.040IN
Connections:
- net 3V3: now also TP17.TESTPOINT; no longer TP17.TP
- net 3V8: now also TP14.TESTPOINT; no longer TP14.TP
- net 5V: now also TP16.TESTPOINT; no longer TP16.TP
- net GND: now also TP15.TESTPOINT; no longer TP15.TP
Changed lines of the file:
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@@
 <part name="TP11" library="testpad" deviceset="TP" device="B1,27"/>
 <part name="TP12" library="testpad" deviceset="TP" device="B1,27"/>
-<part name="TP15" library="testpad" deviceset="PTR1" device="PAD1-13" value="PTR1PAD1-13"/>
-<part name="TP16" library="testpad" deviceset="PTR1" device="PAD1-13" value="PTR1PAD1-13"/>
-<part name="TP14" library="testpad" deviceset="PTR1" device="PAD1-13" value="PTR1PAD1-13"/>
-<part name="TP17" library="testpad" deviceset="PTR1" device="PAD1-13" value="PTR1PAD1-13"/>
 <part name="U$1" library="logos" deviceset="UCB_CAL" device="100MIL"/>
 <part name="GND29" library="umich" deviceset="GND" device=""/>
@@
 <part name="TP5" library="testpad" deviceset="TP" device="B1,27"/>
 <part name="TP13" library="testpad" deviceset="TP" device="B1,27"/>
+<part name="TP17" library="headers" deviceset="TEST_POINT_0.040IN" device=""/>
+<part name="TP14" library="headers" deviceset="TEST_POINT_0.040IN" device=""/>
+<part name="TP15" library="headers" deviceset="TEST_POINT_0.040IN" device=""/>
+<part name="TP16" library="headers" deviceset="TEST_POINT_0.040IN" device=""/>
 </parts>
 <sheets>
@@
 <instance part="R22" gate="G$1" x="187.96" y="50.8" rot="R90"/>
 <instance part="R23" gate="G$1" x="195.58" y="50.8" rot="R90"/>
-<instance part="TP15" gate="G$1" x="78.74" y="101.6" smashed="yes">
-<attribute name="TP_SIGNAL_NAME" x="80.01" y="99.06" size="1.778" layer="97"/>
-</instance>
-<instance part="TP16" gate="G$1" x="22.86" y="129.54" smashed="yes" rot="R180">
-<attribute name="TP_SIGNAL_NAME" x="21.59" y="132.08" size="1.778" layer="97" rot="R180"/>
-</instance>
-<instance part="TP14" gate="G$1" x="96.52" y="129.54" smashed="yes" rot="R180">
-<attribute name="TP_SIGNAL_NAME" x="95.25" y="132.08" size="1.778" layer="97" rot="R180"/>
-</instance>
-<instance part="TP17" gate="G$1" x="96.52" y="175.26" smashed="yes" rot="R180">
-<attribute name="TP_SIGNAL_NAME" x="95.25" y="177.8" size="1.778" layer="97" rot="R180"/>
-</instance>
+<instance part="TP17" gate="G$1" x="96.52" y="175.26" smashed="yes" rot="R270"/>
+<instance part="TP14" gate="G$1" x="96.52" y="129.54" smashed="yes" rot="R270"/>
+<instance part="TP15" gate="G$1" x="81.28" y="101.6" smashed="yes" rot="R90"/>
+<instance part="TP16" gate="G$1" x="20.32" y="129.54" smashed="yes" rot="R270"/>
 </instances>
 <busses>
@@
 <junction x="66.04" y="101.6"/>
 <pinref part="R38" gate="G$1" pin="1"/>
-<wire x1="66.04" y1="104.14" x2="78.74" y2="104.14" width="0.1524" layer="91"/>
 <junction x="66.04" y="104.14"/>
 <pinref part="C26" gate="G$1" pin="1"/>
-<wire x1="78.74" y1="104.14" x2="91.44" y2="104.14" width="0.1524" layer="91"/>
+<wire x1="66.04" y1="104.14" x2="81.28" y2="104.14" width="0.1524" layer="91"/>
+<wire x1="81.28" y1="104.14" x2="91.44" y2="104.14" width="0.1524" layer="91"/>
 <wire x1="104.14" y1="111.76" x2="104.14" y2="104.14" width="0.1524" layer="91"/>
 <wire x1="104.14" y1="104.14" x2="91.44" y2="104.14" width="0.1524" layer="91"/>
 <junction x="91.44" y="104.14"/>
-<pinref part="TP15" gate="G$1" pin="TP"/>
-<junction x="78.74" y="104.14"/>
+<pinref part="TP15" gate="G$1" pin="TESTPOINT"/>
+<junction x="81.28" y="104.14"/>
 </segment>
 <segment>
@@
 <wire x1="7.62" y1="127" x2="15.24" y2="127" width="0.1524" layer="91"/>
 <pinref part="C13" gate="G$1" pin="1"/>
-<wire x1="15.24" y1="127" x2="22.86" y2="127" width="0.1524" layer="91"/>
-<wire x1="22.86" y1="127" x2="27.94" y2="127" width="0.1524" layer="91"/>
+<wire x1="15.24" y1="127" x2="20.32" y2="127" width="0.1524" layer="91"/>
+<wire x1="20.32" y1="127" x2="27.94" y2="127" width="0.1524" layer="91"/>
 <wire x1="15.24" y1="121.92" x2="15.24" y2="127" width="0.1524" layer="91"/>
 <junction x="15.24" y="127"/>
@@
 <junction x="7.62" y="127"/>
 <label x="7.62" y="129.54" size="1.27" layer="95" rot="R90" xref="yes"/>
-<pinref part="TP16" gate="G$1" pin="TP"/>
-<junction x="22.86" y="127"/>
+<pinref part="TP16" gate="G$1" pin="TESTPOINT"/>
+<junction x="20.32" y="127"/>
 </segment>
 </net>
@@
 <junction x="104.14" y="172.72"/>
 <label x="104.14" y="175.26" size="1.27" layer="95" rot="R90" xref="yes"/>
-<pinref part="TP17" gate="G$1" pin="TP"/>
+<pinref part="TP17" gate="G$1" pin="TESTPOINT"/>
 <junction x="96.52" y="172.72"/>
 </segment>
@@
 <junction x="104.14" y="127"/>
 <label x="104.14" y="129.54" size="1.27" layer="95" rot="R90" xref="yes"/>
-<pinref part="TP14" gate="G$1" pin="TP"/>
+<pinref part="TP14" gate="G$1" pin="TESTPOINT"/>
 <junction x="96.52" y="127"/>
 </segment>
@@
 <wire x1="124.46" y1="83.82" x2="111.76" y2="83.82" width="0.1524" layer="91"/>
 <wire x1="111.76" y1="83.82" x2="111.76" y2="86.36" width="0.1524" layer="91"/>
+<pinref part="JP1" gate="G$1" pin="1"/>
 <wire x1="111.76" y1="86.36" x2="81.28" y2="86.36" width="0.1524" layer="91"/>
-<pinref part="JP1" gate="G$1" pin="1"/>
 <wire x1="81.28" y1="86.36" x2="55.88" y2="86.36" width="0.1524" layer="91"/>
 <wire x1="81.28" y1="83.82" x2="81.28" y2="86.36" width="0.1524" layer="91"/>
